File: BeamBuddy/BeamBuddy.sch (KiCad schematic (older format))
At the start: 47 parts, among them J1 DOOR, J10 EXP2, J11 LASER_POT, J2 FLOW, J3 LIM_MIN, J4 12V_TERM, J5 PJ-202AH, J6 TEMP_DISABLE, J7 WP_OUT, J8 TEMP_SENSE, J9 EXP1, U1 MC7805CDTRKG, U2 SN74AHCT14D, U3 CD4082BM96

Commit message: Now with full DigiKey PNs
Parts:
- C1: DK_PN (none) -> 1276-6736-1-ND; SK_PN 1276-6736-1-ND -> (none)
- D1, D2, D3, D4, D5, D6, D7: DK_PN (none) -> 732-4986-1-ND
- D10, D11, D12, D13, D8, D9: DK_PN (none) -> 732-4984-1-ND
- R1, R2, R3, R5: DK_PN (none) -> 311-10.0KHRCT-ND; MPN (none) -> RC0603FR-0710KL
- R10, R11, R12, R13, R14, R15, R16, R17, R18, R9: DK_PN (none) -> 311-560HRCT-ND; MPN (none) -> RC0603FR-07560RL
- R6: DK_PN (none) -> 311-4.70KHRCT-ND; MPN (none) -> RC0603FR-074K7L
- U1: DK_PN (none) -> MC7805CDTRKGOSCT-ND
- U2: MK_PN (none) -> 296-1474-5-ND; MPN (none) -> SN74AHCT14D
- U3: DK_PN (none) -> 296-31523-1-ND; MPN (none) -> CD4082BM96
Changed lines of the file:
@@
 F 2 "OPL_Resistor:R0603" V 2080 1350 50  0001 C CNN
 F 3 "~" H 2150 1350 50  0001 C CNN
+F 4 "RC0603FR-0710KL" H 2150 1350 50  0001 C CNN "MPN"
+F 5 "311-10.0KHRCT-ND" H 2150 1350 50  0001 C CNN "DK_PN"
 	1    2150 1350
 	1    0    0    -1
@@
 F 2 "OPL_Resistor:R0603" V 2380 1350 50  0001 C CNN
 F 3 "~" H 2450 1350 50  0001 C CNN
+F 4 "RC0603FR-0710KL" H 2450 1350 50  0001 C CNN "MPN"
+F 5 "311-10.0KHRCT-ND" H 2450 1350 50  0001 C CNN "DK_PN"
 	1    2450 1350
 	1    0    0    -1
@@
 F 2 "OPL_Resistor:R0603" V 2680 1350 50  0001 C CNN
 F 3 "~" H 2750 1350 50  0001 C CNN
+F 4 "RC0603FR-0710KL" H 2750 1350 50  0001 C CNN "MPN"
+F 5 "311-10.0KHRCT-ND" H 2750 1350 50  0001 C CNN "DK_PN"
 	1    2750 1350
 	1    0    0    -1
@@
 F 2 "CD4082BM96:CD4082BM96" H 6350 1790 60  0001 C CNN
 F 3 "" H 5250 1550 60  0000 C CNN
+F 4 "CD4082BM96" V 5250 1550 50  0001 C CNN "MPN"
+F 5 "296-31523-1-ND" V 5250 1550 50  0001 C CNN "DK_PN"
 	1    5250 1550
 	0    1    1    0
@@
 F 2 "OPL_Resistor:R0603" V 6580 950 50  0001 C CNN
 F 3 "~" H 6650 950 50  0001 C CNN
+F 4 "311-4.70KHRCT-ND" H 6650 950 50  0001 C CNN "DK_PN"
+F 5 "RC0603FR-074K7L" H 6650 950 50  0001 C CNN "MPN"
 	1    6650 950
 	1    0    0    -1
@@
 F 2 "SN74AHCT14D:SN74AHCT14D" H 5000 5140 60  0001 C CNN
 F 3 "" H 3900 4900 60  0000 C CNN
+F 4 "SN74AHCT14D" H 3900 4900 50  0001 C CNN "MPN"
+F 5 "296-1474-5-ND" H 3900 4900 50  0001 C CNN "MK_PN"
 	1    3900 4900
 	1    0    0    -1
@@
 F 3 "" H 7300 3450 50  0001 C CNN
 F 4 "150080VS75000" H 7300 3450 50  0001 C CNN "MPN"
+F 5 "732-4986-1-ND" H 7300 3450 50  0001 C CNN "DK_PN"
 	1    7300 3450
 	-1   0    0    1
@@
 F 3 "~" H 7700 3450 50  0001 C CNN
 F 4 "150080RS75000" H 7700 3450 50  0001 C CNN "MPN"
+F 5 "732-4984-1-ND" H 7700 3450 50  0001 C CNN "DK_PN"
 	1    7700 3450
 	-1   0    0    1
@@
 F 2 "OPL_Resistor:R0603" V 7930 3450 50  0001 C CNN
 F 3 "~" H 8000 3450 50  0001 C CNN
+F 4 "311-560HRCT-ND" H 7000 3900 50  0001 C CNN "DK_PN"
+F 5 "RC0603FR-07560RL" H 7000 3900 50  0001 C CNN "MPN"
 	1    8000 3450
 	0    -1   -1   0
@@
 F 2 "OPL_Resistor:R0603" V 6930 4350 50  0001 C CNN
 F 3 "~" H 7000 4350 50  0001 C CNN
+F 4 "311-560HRCT-ND" H 7000 3900 50  0001 C CNN "DK_PN"
+F 5 "RC0603FR-07560RL" H 7000 3900 50  0001 C CNN "MPN"
 	1    7000 4350
 	0    -1   -1   0
@@
 F 2 "OPL_Resistor:R0603" V 6930 4800 50  0001 C CNN
 F 3 "~" H 7000 4800 50  0001 C CNN
+F 4 "311-560HRCT-ND" H 7000 3900 50  0001 C CNN "DK_PN"
+F 5 "RC0603FR-07560RL" H 7000 3900 50  0001 C CNN "MPN"
 	1    7000 4800
 	0    -1   -1   0
@@
 F 2 "OPL_Resistor:R0603" V 6930 5250 50  0001 C CNN
 F 3 "~" H 7000 5250 50  0001 C CNN
+F 4 "311-560HRCT-ND" H 7000 3900 50  0001 C CNN "DK_PN"
+F 5 "RC0603FR-07560RL" H 7000 3900 50  0001 C CNN "MPN"
 	1    7000 5250
 	0    -1   -1   0
@@
 F 2 "OPL_Resistor:R0603" V 6930 5700 50  0001 C CNN
 F 3 "~" H 7000 5700 50  0001 C CNN
+F 4 "311-560HRCT-ND" H 7000 3900 50  0001 C CNN "DK_PN"
+F 5 "RC0603FR-07560RL" H 7000 3900 50  0001 C CNN "MPN"
 	1    7000 5700
 	0    -1   -1   0
@@
 F 3 "" H 2150 4250 50  0001 C CNN
 F 4 "MC7805CDTRKG" H 2150 4300 50  0001 C CNN "MPN"
+F 5 "MC7805CDTRKGOSCT-ND" H 2150 4300 50  0001 C CNN "DK_PN"
 	1    2150 4300
 	1    0    0    -1
@@
 F 3 "" H 1750 4450 50  0001 C CNN
 F 4 "CL31A106MBHNNNE" H 1780 4600 20  0001 C CNN "MPN"
-F 5 "1276-6736-1-ND" H 1780 4600 20  0001 C CNN "SK_PN"
+F 5 "1276-6736-1-ND" H 1780 4600 20  0001 C CNN "DK_PN"
 	1    1750 4450
 	-1   0    0    -1
@@
 F 3 "" H 2450 4750 50  0001 C CNN
 F 4 "150080VS75000" H 2480 4900 20  0001 C CNN "MPN"
+F 5 "732-4986-1-ND" H 7300 3450 50  0001 C CNN "DK_PN"
 	1    2450 4750
 	-1   0    0    1
@@
 F 2 "OPL_Resistor:R0603" V 6080 5650 50  0001 C CNN
 F 3 "~" H 6150 5650 50  0001 C CNN
+F 4 "RC0603FR-0710KL" H 6150 5650 50  0001 C CNN "MPN"
+F 5 "311-10.0KHRCT-ND" H 6150 5650 50  0001 C CNN "DK_PN"
 	1    6150 5650
 	1    0    0    -1
@@
 F 3 "~" H 7700 3900 50  0001 C CNN
 F 4 "150080RS75000" H 7700 3900 50  0001 C CNN "MPN"
+F 5 "732-4984-1-ND" H 7700 3450 50  0001 C CNN "DK_PN"
 	1    7700 3900
 	-1   0    0    1
@@
 F 3 "~" H 7700 4350 50  0001 C CNN
 F 4 "150080RS75000" H 7700 4350 50  0001 C CNN "MPN"
+F 5 "732-4984-1-ND" H 7700 3450 50  0001 C CNN "DK_PN"
 	1    7700 4350
 	-1   0    0    1
@@
 F 3 "~" H 7700 4800 50  0001 C CNN
 F 4 "150080RS75000" H 7700 4800 50  0001 C CNN "MPN"
+F 5 "732-4984-1-ND" H 7700 3450 50  0001 C CNN "DK_PN"
 	1    7700 4800
 	-1   0    0    1
@@
 F 3 "~" H 7700 5250 50  0001 C CNN
 F 4 "150080RS75000" H 7700 5250 50  0001 C CNN "MPN"
+F 5 "732-4984-1-ND" H 7700 3450 50  0001 C CNN "DK_PN"
 	1    7700 5250
 	-1   0    0    1
@@
 F 3 "~" H 7700 5700 50  0001 C CNN
 F 4 "150080RS75000" H 7700 5700 50  0001 C CNN "MPN"
+F 5 "732-4984-1-ND" H 7700 3450 50  0001 C CNN "DK_PN"
 	1    7700 5700
 	-1   0    0    1
@@
 F 3 "" H 7300 3900 50  0001 C CNN
 F 4 "150080VS75000" H 7300 3900 50  0001 C CNN "MPN"
+F 5 "732-4986-1-ND" H 7300 3450 50  0001 C CNN "DK_PN"
 	1    7300 3900
 	-1   0    0    1
@@
 F 3 "" H 7300 4350 50  0001 C CNN
 F 4 "150080VS75000" H 7300 4350 50  0001 C CNN "MPN"
+F 5 "732-4986-1-ND" H 7300 3450 50  0001 C CNN "DK_PN"
 	1    7300 4350
 	-1   0    0    1
@@
 F 3 "" H 7300 4800 50  0001 C CNN
 F 4 "150080VS75000" H 7300 4800 50  0001 C CNN "MPN"
+F 5 "732-4986-1-ND" H 7300 3450 50  0001 C CNN "DK_PN"
 	1    7300 4800
 	-1   0    0    1
@@
 F 3 "" H 7300 5250 50  0001 C CNN
 F 4 "150080VS75000" H 7300 5250 50  0001 C CNN "MPN"
+F 5 "732-4986-1-ND" H 7300 3450 50  0001 C CNN "DK_PN"
 	1    7300 5250
 	-1   0    0    1
@@
 F 3 "" H 7300 5700 50  0001 C CNN
 F 4 "150080VS75000" H 7300 5700 50  0001 C CNN "MPN"
+F 5 "732-4986-1-ND" H 7300 3450 50  0001 C CNN "DK_PN"
 	1    7300 5700
 	-1   0    0    1
@@
 F 2 "OPL_Resistor:R0603" V 7930 3900 50  0001 C CNN
 F 3 "~" H 8000 3900 50  0001 C CNN
+F 4 "311-560HRCT-ND" H 7000 3900 50  0001 C CNN "DK_PN"
+F 5 "RC0603FR-07560RL" H 7000 3900 50  0001 C CNN "MPN"
 	1    8000 3900
 	0    -1   -1   0
@@
 F 2 "OPL_Resistor:R0603" V 7930 4350 50  0001 C CNN
 F 3 "~" H 8000 4350 50  0001 C CNN
+F 4 "311-560HRCT-ND" H 7000 3900 50  0001 C CNN "DK_PN"
+F 5 "RC0603FR-07560RL" H 7000 3900 50  0001 C CNN "MPN"
 	1    8000 4350
 	0    -1   -1   0
@@
 F 2 "OPL_Resistor:R0603" V 7930 4800 50  0001 C CNN
 F 3 "~" H 8000 4800 50  0001 C CNN
+F 4 "311-560HRCT-ND" H 7000 3900 50  0001 C CNN "DK_PN"
+F 5 "RC0603FR-07560RL" H 7000 3900 50  0001 C CNN "MPN"
 	1    8000 4800
 	0    -1   -1   0
@@
 F 2 "OPL_Resistor:R0603" V 7930 5250 50  0001 C CNN
 F 3 "~" H 8000 5250 50  0001 C CNN
+F 4 "311-560HRCT-ND" H 7000 3900 50  0001 C CNN "DK_PN"
+F 5 "RC0603FR-07560RL" H 7000 3900 50  0001 C CNN "MPN"
 	1    8000 5250
 	0    -1   -1   0
@@
 F 2 "OPL_Resistor:R0603" V 7930 5700 50  0001 C CNN
 F 3 "~" H 8000 5700 50  0001 C CNN
+F 4 "311-560HRCT-ND" H 7000 3900 50  0001 C CNN "DK_PN"
+F 5 "RC0603FR-07560RL" H 7000 3900 50  0001 C CNN "MPN"
 	1    8000 5700
 	0    -1   -1   0
